Commit message: Added the gripper to the urdf

File: urdfs/ur_t42.urdf (robot description, URDF)
Before this commit: robot ur3, 19 links, 18 joints
Links:
- added link flange
- link t42_base_link: geometry collision mesh filename=/home/ubb/Documents/VR_galactic/src/t42_gripper/t42_gripper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 scale=0.1 0.1 0.1; visual mesh filename=/home/ubb/Documents/VR_galactic/src/t42_gripper/t42_gripper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 scale=0.1 0.1 0.1
Joints:
- removed joint wrist_3_link-tool0_fixed_joint
- added joint flange-tool0: type fixed, parent flange, child tool0, origin xyz=0 0 0 rpy=1.5707963267948966 0 1.5707963267948966
- added joint wrist_3-flange: type fixed, parent wrist_3_link, child flange, origin xyz=0 0 0 rpy=0 -1.5707963267948966 -1.5707963267948966

Commit message: Add rmp control for ur

File: urdfs/ur_t42.urdf (robot description, URDF)
Before this commit: robot ur3, 20 links, 19 joints
Links:
- link finger_1_1: geometry collision mesh filename=/home/ubb/Documents/t42_gripper/src/t42_gripper_description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 scale=0.025400 0.025400 0.025400; visual mesh filename=/home/ubb/Documents/t42_gripper/src/t42_gripper_description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 scale=0.025400 0.025400 0.025400
- link finger_1_2: geometry collision mesh filename=/home/ubb/Documents/t42_gripper/src/t42_gripper_description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 scale=0.001 0.001 0.001; visual mesh filename=/home/ubb/Documents/t42_gripper/src/t42_gripper_description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 scale=0.001 0.001 0.001
- link finger_2_1: geometry collision mesh filename=/home/ubb/Documents/t42_gripper/src/t42_gripper_description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 scale=0.025400 0.025400 0.025400; visual mesh filename=/home/ubb/Documents/t42_gripper/src/t42_gripper_description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 scale=0.025400 0.025400 0.025400
- link finger_2_2: geometry collision mesh filename=/home/ubb/Documents/t42_gripper/src/t42_gripper_description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 scale=0.001 0.001 0.001; visual mesh filename=/home/ubb/Documents/t42_gripper/src/t42_gripper_description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 scale=0.001 0.001 0.001
- link swivel_1: geometry collision mesh filename=/home/ubb/Documents/t42_gripper/src/t42_gripper_description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 scale=0.001 0.001 0.001; visual mesh filename=/home/ubb/Documents/t42_gripper/src/t42_gripper_description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 scale=0.001 0.001 0.001
- link swivel_2: geometry collision mesh filename=/home/ubb/Documents/t42_gripper/src/t42_gripper_description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 scale=0.001 0.001 0.001; visual mesh filename=/home/ubb/Documents/t42_gripper/src/t42_gripper_description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 scale=0.001 0.001 0.001
- link t42_base_link: geometry collision mesh filename=/home/ubb/Documents/t42_gripper/src/t42_gripper_description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 scale=1 1 1; visual mesh filename=/home/ubb/Documents/t42_gripper/src/t42_gripper_description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 scale=1 1 1
Joints:
- removed joint base_link-base_fixed_joint
- removed joint base_link-base_link_inertia
- removed joint flange-tool0
- removed joint wrist_3-flange
- removed joint wrist_3_link-ee_link
- added joint base_link_base_fixed_joint: type fixed, parent base_link, child base, origin xyz=0 0 0 rpy=0 0 3.141592653589793
- added joint base_link_base_link_inertia: type fixed, parent base_link, child base_link_inertia, origin xyz=0 0 0 rpy=0 0 3.141592653589793
- added joint flange_tool0: type fixed, parent flange, child tool0, origin xyz=0 0 0 rpy=1.5707963267948966 0 1.5707963267948966
- added joint wrist_3_flange: type fixed, parent wrist_3_link, child flange, origin xyz=0 0 0 rpy=0 -1.5707963267948966 -1.5707963267948966
- added joint wrist_3_link_ee_link: type fixed, parent wrist_3_link, child ee_link, origin xyz=0 0 0 rpy=3.141592653589793 0 0
